Commit message: fix IRB 4600 colors: visual abb_white, collision abb_yellow

File: abb_irb4600_support/urdf/irb4600_20_250_macro.xacro (robot description, xacro)
@@ -9,5 +9,5 @@
           <mesh filename="package://abb_irb4600_support/meshes/irb4600/collision/base_link.stl"/>
         </geometry>
-        <xacro:material_abb_white/>
+        <xacro:material_abb_yellow/>
       </collision>
       <visual name="visual">
@@ -16,7 +16,4 @@
         </geometry>
         <xacro:material_abb_white/>
-        <material name="yellow">
-          <color rgba="1 1 0 1"/>
-        </material>
       </visual>
     </link>
@@ -26,5 +23,5 @@
           <mesh filename="package://abb_irb4600_support/meshes/irb4600/collision/link_1.stl"/>
         </geometry>
-        <xacro:material_abb_white/>
+        <xacro:material_abb_yellow/>
       </collision>
       <visual name="visual">
@@ -33,5 +30,4 @@
         </geometry>
         <xacro:material_abb_white/>
-        <material name="yellow"/>
       </visual>
     </link>
@@ -41,5 +37,5 @@
           <mesh filename="package://abb_irb4600_support/meshes/irb4600_20_250/collision/link_2.stl"/>
         </geometry>
-        <xacro:material_abb_white/>
+        <xacro:material_abb_yellow/>
       </collision>
       <visual name="visual">
@@ -48,5 +44,4 @@
         </geometry>
         <xacro:material_abb_white/>
-        <material name="yellow"/>
       </visual>
     </link>
@@ -56,5 +51,5 @@
           <mesh filename="package://abb_irb4600_support/meshes/irb4600_20_250/collision/link_3.stl"/>
         </geometry>
-        <xacro:material_abb_white/>
+        <xacro:material_abb_yellow/>
       </collision>
       <visual name="visual">
@@ -63,5 +58,4 @@
         </geometry>
         <xacro:material_abb_white/>
-        <material name="yellow"/>
       </visual>
     </link>
@@ -71,5 +65,5 @@
           <mesh filename="package://abb_irb4600_support/meshes/irb4600_20_250/collision/link_4.stl"/>
         </geometry>
-        <xacro:material_abb_white/>
+        <xacro:material_abb_yellow/>
       </collision>
       <visual name="visual">
@@ -78,5 +72,4 @@
         </geometry>
         <xacro:material_abb_white/>
-        <material name="yellow"/>
       </visual>
     </link>
@@ -86,5 +79,5 @@
           <mesh filename="package://abb_irb4600_support/meshes/irb4600_20_250/collision/link_5.stl"/>
         </geometry>
-        <xacro:material_abb_white/>
+        <xacro:material_abb_yellow/>
       </collision>
       <visual name="visual">
@@ -93,5 +86,4 @@
         </geometry>
         <xacro:material_abb_white/>
-        <material name="yellow"/>
       </visual>
     </link>
@@ -101,5 +93,5 @@
           <mesh filename="package://abb_irb4600_support/meshes/irb4600_20_250/collision/link_6.stl"/>
         </geometry>
-        <xacro:material_abb_white/>
+        <xacro:material_abb_yellow/>
       </collision>
       <visual name="visual">
@@ -108,5 +100,4 @@
         </geometry>
         <xacro:material_abb_white/>
-        <material name="yellow"/>
       </visual>
     </link>

File: abb_irb4600_support/urdf/irb4600_40_255_macro.xacro (robot description, xacro)
@@ -9,5 +9,5 @@
           <mesh filename="package://abb_irb4600_support/meshes/irb4600/collision/base_link.stl"/>
         </geometry>
-        <xacro:material_abb_white/>
+        <xacro:material_abb_yellow/>
       </collision>
       <visual name="visual">
@@ -16,7 +16,4 @@
         </geometry>
         <xacro:material_abb_white/>
-        <material name="yellow">
-          <color rgba="1 1 0 1"/>
-        </material>
       </visual>
     </link>
@@ -26,5 +23,5 @@
           <mesh filename="package://abb_irb4600_support/meshes/irb4600/collision/link_1.stl"/>
         </geometry>
-        <xacro:material_abb_white/>
+        <xacro:material_abb_yellow/>
       </collision>
       <visual name="visual">
@@ -33,5 +30,4 @@
         </geometry>
         <xacro:material_abb_white/>
-        <material name="yellow"/>
       </visual>
     </link>
@@ -41,5 +37,5 @@
           <mesh filename="package://abb_irb4600_support/meshes/irb4600_40_255/collision/link_2.stl"/>
         </geometry>
-        <xacro:material_abb_white/>
+        <xacro:material_abb_yellow/>
       </collision>
       <visual name="visual">
@@ -48,5 +44,4 @@
         </geometry>
         <xacro:material_abb_white/>
-        <material name="yellow"/>
       </visual>
     </link>
@@ -56,5 +51,5 @@
           <mesh filename="package://abb_irb4600_support/meshes/irb4600_40_255/collision/link_3.stl"/>
         </geometry>
-        <xacro:material_abb_white/>
+        <xacro:material_abb_yellow/>
       </collision>
       <visual name="visual">
@@ -63,5 +58,4 @@
         </geometry>
         <xacro:material_abb_white/>
-        <material name="yellow"/>
       </visual>
     </link>
@@ -71,5 +65,5 @@
           <mesh filename="package://abb_irb4600_support/meshes/irb4600_40_255/collision/link_4.stl"/>
         </geometry>
-        <xacro:material_abb_white/>
+        <xacro:material_abb_yellow/>
       </collision>
       <visual name="visual">
@@ -78,5 +72,4 @@
         </geometry>
         <xacro:material_abb_white/>
-        <material name="yellow"/>
       </visual>
     </link>
@@ -86,5 +79,5 @@
           <mesh filename="package://abb_irb4600_support/meshes/irb4600_40_255/collision/link_5.stl"/>
         </geometry>
-        <xacro:material_abb_white/>
+        <xacro:material_abb_yellow/>
       </collision>
       <visual name="visual">
@@ -93,5 +86,4 @@
         </geometry>
         <xacro:material_abb_white/>
-        <material name="yellow"/>
       </visual>
     </link>
@@ -101,5 +93,5 @@
           <mesh filename="package://abb_irb4600_support/meshes/irb4600_40_255/collision/link_6.stl"/>
         </geometry>
-        <xacro:material_abb_white/>
+        <xacro:material_abb_yellow/>
       </collision>
       <visual name="visual">
@@ -108,5 +100,4 @@
         </geometry>
         <xacro:material_abb_white/>
-        <material name="yellow"/>
       </visual>
     </link>

File: abb_irb4600_support/urdf/irb4600_60_205_macro.xacro (robot description, xacro)
@@ -2,4 +2,5 @@
 <robot xmlns:xacro="http://ros.org/wiki/xacro">
   <xacro:macro name="abb_irb4600_60_205" params="prefix">
+    <xacro:include filename="$(find abb_resources)/urdf/common_materials.xacro"/>
     <!-- link list -->
     <link name="${prefix}base_link">
@@ -8,4 +9,5 @@
           <mesh filename="package://abb_irb4600_support/meshes/irb4600/collision/base_link.stl"/>
         </geometry>
+        <xacro:material_abb_yellow/>
       </collision>
       <visual name="visual">
@@ -13,7 +15,5 @@
           <mesh filename="package://abb_irb4600_support/meshes/irb4600/visual/base_link.dae"/>
         </geometry>
-        <material name="yellow">
-          <color rgba="1 1 0 1"/>
-        </material>
+        <xacro:material_abb_white/>
       </visual>
     </link>
@@ -23,4 +23,5 @@
           <mesh filename="package://abb_irb4600_support/meshes/irb4600/collision/link_1.stl"/>
         </geometry>
+        <xacro:material_abb_yellow/>
       </collision>
       <visual name="visual">
@@ -28,5 +29,5 @@
           <mesh filename="package://abb_irb4600_support/meshes/irb4600/visual/link_1.dae"/>
         </geometry>
-        <material name="yellow"/>
+        <xacro:material_abb_white/>
       </visual>
     </link>
@@ -36,4 +37,5 @@
           <mesh filename="package://abb_irb4600_support/meshes/irb4600_60_205/collision/link_2.stl"/>
         </geometry>
+        <xacro:material_abb_yellow/>
       </collision>
       <visual name="visual">
@@ -41,5 +43,5 @@
           <mesh filename="package://abb_irb4600_support/meshes/irb4600_60_205/visual/link_2.dae"/>
         </geometry>
-        <material name="yellow"/>
+        <xacro:material_abb_white/>
       </visual>
     </link>
@@ -49,4 +51,5 @@
           <mesh filename="package://abb_irb4600_support/meshes/irb4600_60_205/collision/link_3.stl"/>
         </geometry>
+        <xacro:material_abb_yellow/>
       </collision>
       <visual name="visual">
@@ -54,5 +57,5 @@
           <mesh filename="package://abb_irb4600_support/meshes/irb4600_60_205/visual/link_3.dae"/>
         </geometry>
-        <material name="yellow"/>
+        <xacro:material_abb_white/>
       </visual>
     </link>
@@ -62,4 +65,5 @@
           <mesh filename="package://abb_irb4600_support/meshes/irb4600_60_205/collision/link_4.stl"/>
         </geometry>
+        <xacro:material_abb_yellow/>
       </collision>
       <visual name="visual">
@@ -67,5 +71,5 @@
           <mesh filename="package://abb_irb4600_support/meshes/irb4600_60_205/visual/link_4.dae"/>
         </geometry>
-        <material name="yellow"/>
+        <xacro:material_abb_white/>
       </visual>
     </link>
@@ -75,4 +79,5 @@
           <mesh filename="package://abb_irb4600_support/meshes/irb4600_60_205/collision/link_5.stl"/>
         </geometry>
+        <xacro:material_abb_yellow/>
       </collision>
       <visual name="visual">
@@ -80,5 +85,5 @@
           <mesh filename="package://abb_irb4600_support/meshes/irb4600_60_205/visual/link_5.dae"/>
         </geometry>
-        <material name="yellow"/>
+        <xacro:material_abb_white/>
       </visual>
     </link>
@@ -88,4 +93,5 @@
           <mesh filename="package://abb_irb4600_support/meshes/irb4600_60_205/collision/link_6.stl"/>
         </geometry>
+        <xacro:material_abb_yellow/>
       </collision>
       <visual name="visual">
@@ -93,5 +99,5 @@
           <mesh filename="package://abb_irb4600_support/meshes/irb4600_60_205/visual/link_6.dae"/>
         </geometry>
-        <material name="yellow"/>
+        <xacro:material_abb_white/>
       </visual>
     </link>
