Commit message: fix: correct joint 6 limits for 5/95 GoFa

File: abb_crb15000_support/urdf/crb15000_5_95_macro.xacro (robot description, xacro)
@@ -137,5 +137,5 @@
       <parent link="${prefix}link_5"/>
       <child link="${prefix}link_6"/>
-      <limit effort="0" lower="${radians(-180)}" upper="${radians(180)}" velocity="${radians(200)}"/>
+      <limit effort="0" lower="${radians(-270)}" upper="${radians(270)}" velocity="${radians(200)}"/>
     </joint>
     <!-- end of joint list -->
