Commit message: [irb2600_12_165] fixed joint limits

File: abb_irb2600_support/urdf/irb2600_12_165_macro.xacro (robot description, xacro)
@@ -124,5 +124,5 @@
       <child link="${prefix}link_2" />
       <axis xyz="0 1 0" />
-      <limit lower="-2.705" upper="1.658" effort="0" velocity="3.054" />
+      <limit lower="-1.658" upper="2.705" effort="0" velocity="3.054" />
     </joint>
     <joint name="${prefix}joint_3" type="revolute">
@@ -131,5 +131,5 @@
       <child link="${prefix}link_3" />
       <axis xyz="0 1 0" />
-      <limit lower="-2.705" upper="1.309" effort="0" velocity="3.054" />
+      <limit lower="-3.14159" upper="1.309" effort="0" velocity="3.054" />
     </joint>
     <joint name="${prefix}joint_4" type="revolute">
